Commit message: update: inertiaa for gazebo

File: 5.urdf/simple_car.urdf (robot description, URDF)
Before this commit: robot two_wheel_car, 7 links, 6 joints
Links:
- link base_link: mass None -> 5.0; geometry collision box size=0.6 0.4 0.2; visual mesh filename=package://simple_car_description/meshes/visual/waffle_base.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 scale=0.002 0.00143 0.00125
- link box_on_top_wheel_link: mass None -> 0.5; geometry collision box size=0.2 0.2 0.2; visual box size=0.2 0.2 0.2
- link front_left_wheel_link: mass None -> 0.5; geometry collision cylinder length=0.05 radius=0.1; visual cylinder length=0.05 radius=0.1
- link front_right_wheel_link: mass None -> 0.5; geometry collision cylinder length=0.05 radius=0.1; visual cylinder length=0.05 radius=0.1
- link rear_left_wheel_link: mass None -> 0.5; geometry collision cylinder length=0.05 radius=0.1; visual cylinder length=0.05 radius=0.1
- link rear_right_wheel_link: mass None -> 0.5; geometry collision cylinder length=0.05 radius=0.1; visual cylinder length=0.05 radius=0.1
- link top_wheel_link: mass None -> 0.5; geometry collision cylinder length=0.05 radius=0.1; visual cylinder length=0.05 radius=0.1
Joints:
- joint wheel_joint: limit lower=-1.57 upper=1.57 effort=100 velocity=10 -> lower=-1.5707963267948966 upper=1.5707963267948966 effort=100 velocity=10

File: 5.urdf/src/simple_car_description/urdf/simple_car.properties.xacro (robot description, xacro)
@@ -4,4 +4,5 @@
     <xacro:property name="base_width" value="0.4" />
     <xacro:property name="base_height" value="0.2" />
+    <xacro:property name="base_mass" value="5.0" />
     <xacro:property name="base_mesh_scale_x" value="0.002" />
     <xacro:property name="base_mesh_scale_y" value="0.00143" />
@@ -11,8 +12,11 @@
     <xacro:property name="wheel_width" value="0.05" />
     <xacro:property name="wheel_x_offset" value="0.2" />
+    <xacro:property name="wheel_mass" value="0.5" />
     <xacro:property name="top_wheel_radius" value="0.1" />
     <xacro:property name="top_wheel_height" value="0.05" />
+    <xacro:property name="top_wheel_mass" value="0.5" />
     <xacro:property name="top_box_length" value="0.2" />
     <xacro:property name="top_box_width" value="0.2" />
     <xacro:property name="top_box_height" value="0.2" />
+    <xacro:property name="top_box_mass" value="0.5" />
 </robot>

File: 5.urdf/src/simple_car_description/urdf/simple_car.urdf (robot description, URDF)
Before this commit: robot two_wheel_car, 7 links, 6 joints
Links:
- link base_link: mass None -> 5.0; geometry collision box size=0.6 0.4 0.2; visual mesh filename=package://simple_car_description/meshes/visual/waffle_base.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 scale=0.002 0.00143 0.00125
- link box_on_top_wheel_link: mass None -> 0.5; geometry collision box size=0.2 0.2 0.2; visual box size=0.2 0.2 0.2
- link front_left_wheel_link: mass None -> 0.5; geometry collision cylinder length=0.05 radius=0.1; visual cylinder length=0.05 radius=0.1
- link front_right_wheel_link: mass None -> 0.5; geometry collision cylinder length=0.05 radius=0.1; visual cylinder length=0.05 radius=0.1
- link rear_left_wheel_link: mass None -> 0.5; geometry collision cylinder length=0.05 radius=0.1; visual cylinder length=0.05 radius=0.1
- link rear_right_wheel_link: mass None -> 0.5; geometry collision cylinder length=0.05 radius=0.1; visual cylinder length=0.05 radius=0.1
- link top_wheel_link: mass None -> 0.5; geometry collision cylinder length=0.05 radius=0.1; visual cylinder length=0.05 radius=0.1

File: 5.urdf/src/simple_car_description/urdf/simple_car.urdf.xacro (robot description, xacro)
@@ -3,4 +3,5 @@
     <xacro:include filename="simple_car.materials.xacro" />
     <xacro:include filename="simple_car.properties.xacro" />
+    <xacro:include filename="simple_car.inertias.xacro" />
     <xacro:include filename="simple_car.wheel.xacro" />
     <!-- ====================== Links ====================== -->
@@ -21,4 +22,7 @@
             <origin xyz="0 0 ${base_height / 2}" rpy="0 0 0" />
         </collision>
+        <xacro:inertial_box mass="${base_mass}" x="${base_length}" y="${base_width}" z="${base_height}">
+            <origin xyz="0 0 ${base_height / 2}" rpy="0 0 0" />
+        </xacro:inertial_box>
     </link>
     <!-- Drive wheels: cylinders are rotated so their axles align with the Y-axis. -->
@@ -41,4 +45,13 @@
             <material name="gray" />
         </visual>
+        <collision>
+            <geometry>
+                <cylinder radius="${top_wheel_radius}" length="${top_wheel_height}" />
+            </geometry>
+            <origin xyz="0 0 ${top_wheel_height / 2}" rpy="0 0 0" />
+        </collision>
+        <xacro:inertial_cylinder mass="${top_wheel_mass}" radius="${top_wheel_radius}" length="${top_wheel_height}">
+            <origin xyz="0 0 ${top_wheel_height / 2}" rpy="0 0 0" />
+        </xacro:inertial_cylinder>
     </link>
     <link name="box_on_top_wheel_link">
@@ -51,4 +64,13 @@
             <material name="blue" />
         </visual>
+        <collision>
+            <geometry>
+                <box size="${top_box_length} ${top_box_width} ${top_box_height}" />
+            </geometry>
+            <origin xyz="0 0 ${top_box_height / 2}" rpy="0 0 0" />
+        </collision>
+        <xacro:inertial_box mass="${top_box_mass}" x="${top_box_length}" y="${top_box_width}" z="${top_box_height}">
+            <origin xyz="0 0 ${top_box_height / 2}" rpy="0 0 0" />
+        </xacro:inertial_box>
     </link>
     <!-- ===================== Joints ====================== -->

File: 5.urdf/src/simple_car_description/urdf/simple_car.wheel.xacro (robot description, xacro)
@@ -10,4 +10,13 @@
                 <material name="gray" />
             </visual>
+            <collision>
+                <geometry>
+                    <cylinder radius="${wheel_radius}" length="${wheel_width}" />
+                </geometry>
+                <origin xyz="0 0 0" rpy="${pi / 2} 0 0" />
+            </collision>
+            <xacro:inertial_cylinder mass="${wheel_mass}" radius="${wheel_radius}" length="${wheel_width}">
+                <origin xyz="0 0 0" rpy="${pi / 2} 0 0" />
+            </xacro:inertial_cylinder>
         </link>
         <joint name="${name}_wheel_joint" type="continuous">

Commit message: update: adjust collision

File: 5.urdf/simple_car.urdf (robot description, URDF)
Before this commit: robot two_wheel_car, 7 links, 6 joints
Links:
- link base_link: geometry collision box size=0.6 0.4 0.15; visual mesh filename=package://simple_car_description/meshes/visual/waffle_base.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 scale=0.002 0.00143 0.00125

File: 5.urdf/src/simple_car_description/urdf/simple_car.properties.xacro (robot description, xacro)
@@ -3,5 +3,5 @@
     <xacro:property name="base_length" value="0.6" />
     <xacro:property name="base_width" value="0.4" />
-    <xacro:property name="base_height" value="0.2" />
+    <xacro:property name="base_height" value="0.15" />
     <xacro:property name="base_mass" value="5.0" />
     <xacro:property name="base_mesh_scale_x" value="0.002" />

File: 5.urdf/src/simple_car_description/urdf/simple_car.urdf (robot description, URDF)
Before this commit: robot two_wheel_car, 7 links, 6 joints
Links:
- link base_link: geometry collision box size=0.6 0.4 0.15; visual mesh filename=package://simple_car_description/meshes/visual/waffle_base.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 scale=0.002 0.00143 0.00125

File: 5.urdf/src/simple_car_description/urdf/simple_car.urdf.xacro (robot description, xacro)
@@ -20,8 +20,8 @@
                 <box size="${base_length} ${base_width} ${base_height}" />
             </geometry>
-            <origin xyz="0 0 ${base_height / 2}" rpy="0 0 0" />
+            <origin xyz="0 0 ${base_mesh_z_offset + base_height / 2}" rpy="0 0 0" />
         </collision>
         <xacro:inertial_box mass="${base_mass}" x="${base_length}" y="${base_width}" z="${base_height}">
-            <origin xyz="0 0 ${base_height / 2}" rpy="0 0 0" />
+            <origin xyz="0 0 ${base_mesh_z_offset + base_height / 2}" rpy="0 0 0" />
         </xacro:inertial_box>
     </link>
@@ -80,5 +80,5 @@
         <child link="top_wheel_link" />
         <!-- Place the platform joint on the top surface of the chassis. -->
-        <origin xyz="0 0 ${base_height}" rpy="0 0 0" />
+        <origin xyz="0 0 ${base_mesh_z_offset + base_height}" rpy="0 0 0" />
         <axis xyz="0 0 1" />
         <limit effort="100" velocity="10" lower="${pi / -2}" upper="${pi / 2}" />

Commit message: update: make bridge between gazebo and ros2 and make robot move

File: 5.urdf/simple_car.urdf (robot description, URDF)
Before this commit: robot two_wheel_car, 7 links, 6 joints
Joints:
- joint front_left_wheel_joint: limit (none) -> effort=100 velocity=10
- joint front_right_wheel_joint: limit (none) -> effort=100 velocity=10
- joint rear_left_wheel_joint: limit (none) -> effort=100 velocity=10
- joint rear_right_wheel_joint: limit (none) -> effort=100 velocity=10

File: 5.urdf/src/simple_car_description/urdf/simple_car.gazebo.xacro (robot description, xacro)
@@ -2,9 +2,9 @@
 <robot xmlns:xacro="http://www.ros.org/wiki/xacro">
     <!-- ================= Gazebo Plugins / Systems ================= -->
-    <!-- Joint State Publisher: Publishes joint states to Gazebo topic so they can be bridged to ROS 2 /joint_states for RViz and robot_state_publisher -->
     <gazebo>
+        <!-- Joint State Publisher: Publishes joint states to Gazebo topic for RViz & robot_state_publisher -->
         <plugin filename="gz-sim-joint-state-publisher-system"
                 name="gz::sim::systems::JointStatePublisher">
-            <topic>joint_states</topic>
+            <topic>/joint_states</topic>
             <joint_name>front_left_wheel_joint</joint_name>
             <joint_name>front_right_wheel_joint</joint_name>
@@ -13,4 +13,28 @@
             <joint_name>wheel_joint</joint_name>
         </plugin>
+        <!-- Differential Drive: Controls wheels via velocity commands (cmd_vel) and publishes odometry -->
+        <plugin filename="gz-sim-diff-drive-system"
+                name="gz::sim::systems::DiffDrive">
+            <!-- Left wheels -->
+            <left_joint>front_left_wheel_joint</left_joint>
+            <left_joint>rear_left_wheel_joint</left_joint>
+            <!-- Right wheels -->
+            <right_joint>front_right_wheel_joint</right_joint>
+            <right_joint>rear_right_wheel_joint</right_joint>
+            <!-- Kinematics -->
+            <wheel_separation>${base_width + wheel_width}</wheel_separation>
+            <wheel_radius>${wheel_radius}</wheel_radius>
+            <!-- Limits & Torque -->
+            <max_linear_acceleration>5.0</max_linear_acceleration>
+            <max_angular_acceleration>5.0</max_angular_acceleration>
+            <max_wheel_torque>50.0</max_wheel_torque>
+            <!-- Topics & Frames (use leading slash to bind to global topics matching ros_gz_bridge) -->
+            <topic>/cmd_vel</topic>
+            <odom_topic>/odom</odom_topic>
+            <tf_topic>/tf</tf_topic>
+            <frame_id>odom</frame_id>
+            <child_frame_id>base_link</child_frame_id>
+            <odom_publish_frequency>50</odom_publish_frequency>
+        </plugin>
     </gazebo>
 </robot>

File: 5.urdf/src/simple_car_description/urdf/simple_car.urdf (robot description, URDF)
Before this commit: robot two_wheel_car, 7 links, 6 joints
Joints:
- joint front_left_wheel_joint: limit (none) -> effort=100 velocity=10
- joint front_right_wheel_joint: limit (none) -> effort=100 velocity=10
- joint rear_left_wheel_joint: limit (none) -> effort=100 velocity=10
- joint rear_right_wheel_joint: limit (none) -> effort=100 velocity=10

File: 5.urdf/src/simple_car_description/urdf/simple_car.wheel.xacro (robot description, xacro)
@@ -16,8 +16,18 @@
                 <origin xyz="0 0 0" rpy="${pi / 2} 0 0" />
             </collision>
-            <xacro:inertial_cylinder mass="${wheel_mass}" radius="${wheel_radius}" length="${wheel_width}">
+            <xacro:inertial_cylinder mass="${wheel_mass}" radius="${wheel_radius}"
+                length="${wheel_width}">
                 <origin xyz="0 0 0" rpy="${pi / 2} 0 0" />
             </xacro:inertial_cylinder>
         </link>
+        <!-- friction -->
+        <gazebo reference="${name}_wheel_link">
+            <mu1>1.0</mu1>
+            <mu2>0.5</mu2>
+            <kp>1000000.0</kp>
+            <kd>100.0</kd>
+            <minDepth>0.001</minDepth>
+            <maxVel>1.0</maxVel>
+        </gazebo>
         <joint name="${name}_wheel_joint" type="continuous">
             <parent link="base_link" />
@@ -25,4 +35,6 @@
             <origin xyz="${x} ${y} ${wheel_radius}" rpy="0 0 0" />
             <axis xyz="0 1 0" />
+            <limit effort="100" velocity="10" />
+            <dynamics damping="0.1" friction="0.1" />
         </joint>
     </xacro:macro>

Commit message: update: add camera sensor

File: 5.urdf/simple_car.urdf (robot description, URDF)
Before this commit: robot two_wheel_car, 7 links, 6 joints
Links:
- added link camera_link, mass 0.05; collision cylinder length=0.04 radius=0.02; visual cylinder length=0.04 radius=0.02
- added link camera_optical_frame
Joints:
- added joint camera_joint: type fixed, parent box_on_top_wheel_link, child camera_link, origin xyz=0.1 0 0.1 rpy=0 0 0
- added joint camera_optical_joint: type fixed, parent camera_link, child camera_optical_frame, origin xyz=0.04 0 0 rpy=-1.5707963267948966 0 -1.5707963267948966

File: 5.urdf/src/simple_car_description/urdf/simple_car.gazebo.xacro (robot description, xacro)
@@ -2,4 +2,26 @@
 <robot xmlns:xacro="http://www.ros.org/wiki/xacro">
     <!-- ================= Gazebo Plugins / Systems ================= -->
+    <gazebo reference="camera_link">
+        <sensor name="camera" type="camera">
+            <always_on>true</always_on>
+            <visualize>true</visualize>
+            <update_rate>30</update_rate>
+            <topic>/camera/image_raw</topic>
+            <gz_frame_id>camera_optical_frame</gz_frame_id>
+            <camera name="camera_sensor">
+                <camera_info_topic>/camera/camera_info</camera_info_topic>
+                <horizontal_fov>1.089</horizontal_fov>
+                <image>
+                    <width>640</width>
+                    <height>480</height>
+                    <format>R8G8B8</format>
+                </image>
+                <clip>
+                    <near>0.05</near>
+                    <far>8.0</far>
+                </clip>
+            </camera>
+        </sensor>
+    </gazebo>
     <gazebo>
         <!-- Joint State Publisher: Publishes joint states to Gazebo topic for RViz & robot_state_publisher -->

File: 5.urdf/src/simple_car_description/urdf/simple_car.materials.xacro (robot description, xacro)
@@ -7,3 +7,6 @@
         <color rgba="0.5 0.5 0.5 1" />
     </material>
+    <material name="black">
+        <color rgba="0.1 0.1 0.1 1" />
+    </material>
 </robot>

File: 5.urdf/src/simple_car_description/urdf/simple_car.properties.xacro (robot description, xacro)
@@ -20,3 +20,6 @@
     <xacro:property name="top_box_height" value="0.2" />
     <xacro:property name="top_box_mass" value="0.5" />
+    <xacro:property name="camera_radius" value="0.02" />
+    <xacro:property name="camera_length" value="0.04" />
+    <xacro:property name="camera_mass" value="0.05" />
 </robot>

File: 5.urdf/src/simple_car_description/urdf/simple_car.urdf (robot description, URDF)
Before this commit: robot two_wheel_car, 7 links, 6 joints
Links:
- added link camera_link, mass 0.05; collision cylinder length=0.04 radius=0.02; visual cylinder length=0.04 radius=0.02
- added link camera_optical_frame
Joints:
- added joint camera_joint: type fixed, parent box_on_top_wheel_link, child camera_link, origin xyz=0.1 0 0.1 rpy=0 0 0
- added joint camera_optical_joint: type fixed, parent camera_link, child camera_optical_frame, origin xyz=0.04 0 0 rpy=-1.5707963267948966 0 -1.5707963267948966

File: 5.urdf/src/simple_car_description/urdf/simple_car.urdf.xacro (robot description, xacro)
@@ -75,4 +75,26 @@
         </xacro:inertial_box>
     </link>
+    <!-- Camera sensor mounted on the front of the top box -->
+    <link name="camera_link">
+        <visual>
+            <geometry>
+                <cylinder radius="${camera_radius}" length="${camera_length}" />
+            </geometry>
+            <!-- Align cylinder along X (forward) and extend outward from mounting surface -->
+            <origin xyz="${camera_length / 2} 0 0" rpy="0 ${pi / 2} 0" />
+            <material name="black" />
+        </visual>
+        <collision>
+            <geometry>
+                <cylinder radius="${camera_radius}" length="${camera_length}" />
+            </geometry>
+            <origin xyz="${camera_length / 2} 0 0" rpy="0 ${pi / 2} 0" />
+        </collision>
+        <xacro:inertial_cylinder mass="${camera_mass}" radius="${camera_radius}" length="${camera_length}">
+            <origin xyz="${camera_length / 2} 0 0" rpy="0 ${pi / 2} 0" />
+        </xacro:inertial_cylinder>
+    </link>
+    <!-- Camera optical frame (REP-103 convention: +Z forward, +X right, +Y down) -->
+    <link name="camera_optical_frame" />
     <!-- ===================== Joints ====================== -->
     <!-- Upper assembly: rotate the platform around Z and rigidly attach its box. -->
@@ -91,3 +113,15 @@
         <origin xyz="0 0 ${top_wheel_height}" rpy="0 0 0" />
     </joint>
+    <joint name="camera_joint" type="fixed">
+        <parent link="box_on_top_wheel_link" />
+        <child link="camera_link" />
+        <!-- Place the camera joint at the front face center of the top box. -->
+        <origin xyz="${top_box_length / 2} 0 ${top_box_height / 2}" rpy="0 0 0" />
+    </joint>
+    <joint name="camera_optical_joint" type="fixed">
+        <parent link="camera_link" />
+        <child link="camera_optical_frame" />
+        <!-- Optical frame transform: +Z forward along camera lens, +X right, +Y down -->
+        <origin xyz="${camera_length} 0 0" rpy="${-pi / 2} 0 ${-pi / 2}" />
+    </joint>
 </robot>

Commit message: update: add 2 part robot arm

File: 5.urdf/simple_car.urdf (robot description, URDF)
Before this commit: robot two_wheel_car, 9 links, 8 joints
Links:
- added link arm_link_1, mass 0.2; collision cylinder length=0.5 radius=0.02; visual cylinder length=0.5 radius=0.02
- added link arm_link_2, mass 0.2; collision cylinder length=0.5 radius=0.02; visual cylinder length=0.5 radius=0.02
Joints:
- added joint arm_joint_1: type revolute, parent box_on_top_wheel_link, child arm_link_1, origin xyz=0 0 0.2 rpy=0 0 0, axis 0 1 0, limit lower=-1.5707963267948966 upper=1.5707963267948966 effort=100 velocity=10
- added joint arm_joint_2: type revolute, parent arm_link_1, child arm_link_2, origin xyz=0 0 0.5 rpy=0 0 0, axis 0 1 0, limit lower=-1.5707963267948966 upper=1.5707963267948966 effort=100 velocity=10

File: 5.urdf/src/simple_car_description/urdf/simple_car.gazebo.xacro (robot description, xacro)
@@ -34,4 +34,6 @@
             <joint_name>rear_right_wheel_joint</joint_name>
             <joint_name>wheel_joint</joint_name>
+            <joint_name>arm_joint_1</joint_name>
+            <joint_name>arm_joint_2</joint_name>
         </plugin>
         <!-- Differential Drive: Controls wheels via velocity commands (cmd_vel) and publishes odometry -->

File: 5.urdf/src/simple_car_description/urdf/simple_car.materials.xacro (robot description, xacro)
@@ -10,3 +10,6 @@
         <color rgba="0.1 0.1 0.1 1" />
     </material>
+    <material name="orange">
+        <color rgba="1.0 0.5 0.0 1.0" />
+    </material>
 </robot>

File: 5.urdf/src/simple_car_description/urdf/simple_car.properties.xacro (robot description, xacro)
@@ -23,3 +23,6 @@
     <xacro:property name="camera_length" value="0.04" />
     <xacro:property name="camera_mass" value="0.05" />
+    <xacro:property name="arm_length" value="0.5" />
+    <xacro:property name="arm_radius" value="0.02" />
+    <xacro:property name="arm_mass" value="0.2" />
 </robot>

File: 5.urdf/src/simple_car_description/urdf/simple_car.urdf (robot description, URDF)
Before this commit: robot two_wheel_car, 9 links, 8 joints
Links:
- added link arm_link_1, mass 0.2; collision cylinder length=0.5 radius=0.02; visual cylinder length=0.5 radius=0.02
- added link arm_link_2, mass 0.2; collision cylinder length=0.5 radius=0.02; visual cylinder length=0.5 radius=0.02
Joints:
- added joint arm_joint_1: type revolute, parent box_on_top_wheel_link, child arm_link_1, origin xyz=0 0 0.2 rpy=0 0 0, axis 0 1 0, limit lower=-1.5707963267948966 upper=1.5707963267948966 effort=100 velocity=10
- added joint arm_joint_2: type revolute, parent arm_link_1, child arm_link_2, origin xyz=0 0 0.5 rpy=0 0 0, axis 0 1 0, limit lower=-1.5707963267948966 upper=1.5707963267948966 effort=100 velocity=10

File: 5.urdf/src/simple_car_description/urdf/simple_car.urdf.xacro (robot description, xacro)
@@ -5,4 +5,5 @@
     <xacro:include filename="simple_car.inertias.xacro" />
     <xacro:include filename="simple_car.wheel.xacro" />
+    <xacro:include filename="simple_car.arm.xacro" />
     <xacro:include filename="simple_car.gazebo.xacro" />
     <!-- ====================== Links ====================== -->
@@ -125,3 +126,5 @@
         <origin xyz="${camera_length} 0 0" rpy="${-pi / 2} 0 ${-pi / 2}" />
     </joint>
+    <!-- 2-part robotic arm mounted above the top box -->
+    <xacro:arm parent="box_on_top_wheel_link" />
 </robot>
