Commit message: update: use xacro constants

File: 5.urdf/src/simple_car_description/urdf/simple_car.urdf.xacro (robot description, xacro)
@@ -8,4 +8,16 @@
         <color rgba="0.5 0.5 0.5 1" />
     </material>
+    <!-- ==================== Dimensions ==================== -->
+    <xacro:property name="base_length" value="0.6" />
+    <xacro:property name="base_width" value="0.4" />
+    <xacro:property name="base_height" value="0.2" />
+    <xacro:property name="wheel_radius" value="0.1" />
+    <xacro:property name="wheel_width" value="0.05" />
+    <xacro:property name="wheel_x_offset" value="0.2" />
+    <xacro:property name="top_wheel_radius" value="0.1" />
+    <xacro:property name="top_wheel_height" value="0.05" />
+    <xacro:property name="top_box_length" value="0.2" />
+    <xacro:property name="top_box_width" value="0.2" />
+    <xacro:property name="top_box_height" value="0.2" />
     <!-- ====================== Links ====================== -->
     <!-- Chassis: 0.6 m long (X), 0.4 m wide (Y), and 0.2 m high (Z). -->
@@ -13,8 +25,8 @@
         <visual>
             <geometry>
-                <box size="0.6 0.4 0.2" />
+                <box size="${base_length} ${base_width} ${base_height}" />
             </geometry>
             <!-- Raise the visual by half its height so the link frame is at ground level. -->
-            <origin xyz="0 0 0.1" rpy="0 0 0" />
+            <origin xyz="0 0 ${base_height / 2}" rpy="0 0 0" />
             <material name="blue" />
         </visual>
@@ -24,5 +36,5 @@
         <visual>
             <geometry>
-                <cylinder radius="0.1" length="0.05" />
+                <cylinder radius="${wheel_radius}" length="${wheel_width}" />
             </geometry>
             <origin xyz="0 0 0" rpy="1.5708 0 0" />
@@ -33,5 +45,5 @@
         <visual>
             <geometry>
-                <cylinder radius="0.1" length="0.05" />
+                <cylinder radius="${wheel_radius}" length="${wheel_width}" />
             </geometry>
             <origin xyz="0 0 0" rpy="1.5708 0 0" />
@@ -42,5 +54,5 @@
         <visual>
             <geometry>
-                <cylinder radius="0.1" length="0.05" />
+                <cylinder radius="${wheel_radius}" length="${wheel_width}" />
             </geometry>
             <origin xyz="0 0 0" rpy="1.5708 0 0" />
@@ -51,5 +63,5 @@
         <visual>
             <geometry>
-                <cylinder radius="0.1" length="0.05" />
+                <cylinder radius="${wheel_radius}" length="${wheel_width}" />
             </geometry>
             <origin xyz="0 0 0" rpy="1.5708 0 0" />
@@ -61,8 +73,8 @@
         <visual>
             <geometry>
-                <cylinder radius="0.1" length="0.05" />
+                <cylinder radius="${top_wheel_radius}" length="${top_wheel_height}" />
             </geometry>
             <!-- Raise the cylinder by half its length above the joint frame. -->
-            <origin xyz="0 0 0.025" rpy="0 0 0" />
+            <origin xyz="0 0 ${top_wheel_height / 2}" rpy="0 0 0" />
             <material name="gray" />
         </visual>
@@ -71,8 +83,8 @@
         <visual>
             <geometry>
-                <box size="0.2 0.2 0.2" />
+                <box size="${top_box_length} ${top_box_width} ${top_box_height}" />
             </geometry>
             <!-- Raise the box by half its height above its link frame. -->
-            <origin xyz="0 0 0.1" rpy="0 0 0" />
+            <origin xyz="0 0 ${top_box_height / 2}" rpy="0 0 0" />
             <material name="blue" />
         </visual>
@@ -83,5 +95,6 @@
         <parent link="base_link" />
         <child link="front_left_wheel_link" />
-        <origin xyz="0.2 0.225 0.1" rpy="0 0 0" />
+        <origin xyz="${wheel_x_offset} ${base_width / 2 + wheel_width / 2} ${wheel_radius}"
+            rpy="0 0 0" />
         <axis xyz="0 1 0" />
     </joint>
@@ -89,5 +102,6 @@
         <parent link="base_link" />
         <child link="front_right_wheel_link" />
-        <origin xyz="0.2 -0.225 0.1" rpy="0 0 0" />
+        <origin xyz="${wheel_x_offset} ${-(base_width / 2 + wheel_width / 2)} ${wheel_radius}"
+            rpy="0 0 0" />
         <axis xyz="0 1 0" />
     </joint>
@@ -95,5 +109,6 @@
         <parent link="base_link" />
         <child link="rear_left_wheel_link" />
-        <origin xyz="-0.2 0.225 0.1" rpy="0 0 0" />
+        <origin xyz="${-wheel_x_offset} ${base_width / 2 + wheel_width / 2} ${wheel_radius}"
+            rpy="0 0 0" />
         <axis xyz="0 1 0" />
     </joint>
@@ -101,5 +116,6 @@
         <parent link="base_link" />
         <child link="rear_right_wheel_link" />
-        <origin xyz="-0.2 -0.225 0.1" rpy="0 0 0" />
+        <origin xyz="${-wheel_x_offset} ${-(base_width / 2 + wheel_width / 2)} ${wheel_radius}"
+            rpy="0 0 0" />
         <axis xyz="0 1 0" />
     </joint>
@@ -109,7 +125,7 @@
         <child link="top_wheel_link" />
         <!-- Place the platform joint on the top surface of the chassis. -->
-        <origin xyz="0 0 0.2" rpy="0 0 0" />
+        <origin xyz="0 0 ${base_height}" rpy="0 0 0" />
         <axis xyz="0 0 1" />
-        <limit effort="100" velocity="10" lower="-1.57" upper="1.57" />
+        <limit effort="100" velocity="10" lower="${pi / -2}" upper="${pi / 2}" />
     </joint>
     <joint name="box_on_wheel_joint" type="fixed">
@@ -117,5 +133,5 @@
         <child link="box_on_top_wheel_link" />
         <!-- Place the box on the top surface of the rotating platform. -->
-        <origin xyz="0 0 0.05" rpy="0 0 0" />
+        <origin xyz="0 0 ${top_wheel_height}" rpy="0 0 0" />
     </joint>
 </robot>

Commit message: update: use macro to reduce duplicated code

File: 5.urdf/src/simple_car_description/urdf/simple_car.urdf.xacro (robot description, xacro)
@@ -20,4 +20,22 @@
     <xacro:property name="top_box_width" value="0.2" />
     <xacro:property name="top_box_height" value="0.2" />
+    <!-- ===================== Macros ====================== -->
+    <xacro:macro name="wheel" params="name x y">
+        <link name="${name}_wheel_link">
+            <visual>
+                <geometry>
+                    <cylinder radius="${wheel_radius}" length="${wheel_width}" />
+                </geometry>
+                <origin xyz="0 0 0" rpy="${pi / 2} 0 0" />
+                <material name="gray" />
+            </visual>
+        </link>
+        <joint name="${name}_wheel_joint" type="continuous">
+            <parent link="base_link" />
+            <child link="${name}_wheel_link" />
+            <origin xyz="${x} ${y} ${wheel_radius}" rpy="0 0 0" />
+            <axis xyz="0 1 0" />
+        </joint>
+    </xacro:macro>
     <!-- ====================== Links ====================== -->
     <!-- Chassis: 0.6 m long (X), 0.4 m wide (Y), and 0.2 m high (Z). -->
@@ -33,40 +51,12 @@
     </link>
     <!-- Drive wheels: cylinders are rotated so their axles align with the Y-axis. -->
-    <link name="front_left_wheel_link">
-        <visual>
-            <geometry>
-                <cylinder radius="${wheel_radius}" length="${wheel_width}" />
-            </geometry>
-            <origin xyz="0 0 0" rpy="1.5708 0 0" />
-            <material name="gray" />
-        </visual>
-    </link>
-    <link name="front_right_wheel_link">
-        <visual>
-            <geometry>
-                <cylinder radius="${wheel_radius}" length="${wheel_width}" />
-            </geometry>
-            <origin xyz="0 0 0" rpy="1.5708 0 0" />
-            <material name="gray" />
-        </visual>
-    </link>
-    <link name="rear_left_wheel_link">
-        <visual>
-            <geometry>
-                <cylinder radius="${wheel_radius}" length="${wheel_width}" />
-            </geometry>
-            <origin xyz="0 0 0" rpy="1.5708 0 0" />
-            <material name="gray" />
-        </visual>
-    </link>
-    <link name="rear_right_wheel_link">
-        <visual>
-            <geometry>
-                <cylinder radius="${wheel_radius}" length="${wheel_width}" />
-            </geometry>
-            <origin xyz="0 0 0" rpy="1.5708 0 0" />
-            <material name="gray" />
-        </visual>
-    </link>
+    <xacro:wheel name="front_left" x="${wheel_x_offset}"
+        y="${base_width / 2 + wheel_width / 2}" />
+    <xacro:wheel name="front_right" x="${wheel_x_offset}"
+        y="${-(base_width / 2 + wheel_width / 2)}" />
+    <xacro:wheel name="rear_left" x="${-wheel_x_offset}"
+        y="${base_width / 2 + wheel_width / 2}" />
+    <xacro:wheel name="rear_right" x="${-wheel_x_offset}"
+        y="${-(base_width / 2 + wheel_width / 2)}" />
     <!-- Upper rotating platform and its mounted box. -->
     <link name="top_wheel_link">
@@ -91,33 +81,4 @@
     </link>
     <!-- ===================== Joints ====================== -->
-    <!-- Wheel axles: X selects front/rear, Y selects left/right, and Z is wheel radius. -->
-    <joint name="front_left_wheel_joint" type="continuous">
-        <parent link="base_link" />
-        <child link="front_left_wheel_link" />
-        <origin xyz="${wheel_x_offset} ${base_width / 2 + wheel_width / 2} ${wheel_radius}"
-            rpy="0 0 0" />
-        <axis xyz="0 1 0" />
-    </joint>
-    <joint name="front_right_wheel_joint" type="continuous">
-        <parent link="base_link" />
-        <child link="front_right_wheel_link" />
-        <origin xyz="${wheel_x_offset} ${-(base_width / 2 + wheel_width / 2)} ${wheel_radius}"
-            rpy="0 0 0" />
-        <axis xyz="0 1 0" />
-    </joint>
-    <joint name="rear_left_wheel_joint" type="continuous">
-        <parent link="base_link" />
-        <child link="rear_left_wheel_link" />
-        <origin xyz="${-wheel_x_offset} ${base_width / 2 + wheel_width / 2} ${wheel_radius}"
-            rpy="0 0 0" />
-        <axis xyz="0 1 0" />
-    </joint>
-    <joint name="rear_right_wheel_joint" type="continuous">
-        <parent link="base_link" />
-        <child link="rear_right_wheel_link" />
-        <origin xyz="${-wheel_x_offset} ${-(base_width / 2 + wheel_width / 2)} ${wheel_radius}"
-            rpy="0 0 0" />
-        <axis xyz="0 1 0" />
-    </joint>
     <!-- Upper assembly: rotate the platform around Z and rigidly attach its box. -->
     <joint name="wheel_joint" type="revolute">

Commit message: update: split urdf file

File: 5.urdf/src/simple_car_description/urdf/simple_car.urdf.xacro (robot description, xacro)
@@ -1,41 +1,7 @@
 <?xml version="1.0"?>
 <robot name="two_wheel_car" xmlns:xacro="http://www.ros.org/wiki/xacro">
-    <!-- ==================== Materials ==================== -->
-    <material name="blue">
-        <color rgba="0.6 0.2 0.6 1" />
-    </material>
-    <material name="gray">
-        <color rgba="0.5 0.5 0.5 1" />
-    </material>
-    <!-- ==================== Dimensions ==================== -->
-    <xacro:property name="base_length" value="0.6" />
-    <xacro:property name="base_width" value="0.4" />
-    <xacro:property name="base_height" value="0.2" />
-    <xacro:property name="wheel_radius" value="0.1" />
-    <xacro:property name="wheel_width" value="0.05" />
-    <xacro:property name="wheel_x_offset" value="0.2" />
-    <xacro:property name="top_wheel_radius" value="0.1" />
-    <xacro:property name="top_wheel_height" value="0.05" />
-    <xacro:property name="top_box_length" value="0.2" />
-    <xacro:property name="top_box_width" value="0.2" />
-    <xacro:property name="top_box_height" value="0.2" />
-    <!-- ===================== Macros ====================== -->
-    <xacro:macro name="wheel" params="name x y">
-        <link name="${name}_wheel_link">
-            <visual>
-                <geometry>
-                    <cylinder radius="${wheel_radius}" length="${wheel_width}" />
-                </geometry>
-                <origin xyz="0 0 0" rpy="${pi / 2} 0 0" />
-                <material name="gray" />
-            </visual>
-        </link>
-        <joint name="${name}_wheel_joint" type="continuous">
-            <parent link="base_link" />
-            <child link="${name}_wheel_link" />
-            <origin xyz="${x} ${y} ${wheel_radius}" rpy="0 0 0" />
-            <axis xyz="0 1 0" />
-        </joint>
-    </xacro:macro>
+    <xacro:include filename="simple_car.materials.xacro" />
+    <xacro:include filename="simple_car.properties.xacro" />
+    <xacro:include filename="simple_car.wheel.xacro" />
     <!-- ====================== Links ====================== -->
     <!-- Chassis: 0.6 m long (X), 0.4 m wide (Y), and 0.2 m high (Z). -->
