Commit message: chore: generate urdf from xacro

File: 5.urdf/src/simple_car_description/urdf/simple_car.urdf (robot description, URDF)
Before this commit: robot two_wheel_car, 7 links, 6 joints
Joints:
- joint wheel_joint: limit lower=-1.57 upper=1.57 effort=100 velocity=10 -> lower=-1.5707963267948966 upper=1.5707963267948966 effort=100 velocity=10
