Commit message: update: use real model mesh

File: 5.urdf/src/simple_car_description/urdf/simple_car.properties.xacro (robot description, xacro)
@@ -4,4 +4,8 @@
     <xacro:property name="base_width" value="0.4" />
     <xacro:property name="base_height" value="0.2" />
+    <xacro:property name="base_mesh_scale_x" value="0.002" />
+    <xacro:property name="base_mesh_scale_y" value="0.00143" />
+    <xacro:property name="base_mesh_scale_z" value="0.00125" />
+    <xacro:property name="base_mesh_z_offset" value="0.05" />
     <xacro:property name="wheel_radius" value="0.1" />
     <xacro:property name="wheel_width" value="0.05" />

File: 5.urdf/src/simple_car_description/urdf/simple_car.urdf.xacro (robot description, xacro)
@@ -5,14 +5,20 @@
     <xacro:include filename="simple_car.wheel.xacro" />
     <!-- ====================== Links ====================== -->
-    <!-- Chassis: 0.6 m long (X), 0.4 m wide (Y), and 0.2 m high (Z). -->
+    <!-- Chassis visual uses an Apache-2.0 TurtleBot3 Waffle base mesh. -->
     <link name="base_link">
         <visual>
             <geometry>
+                <mesh filename="package://simple_car_description/meshes/visual/waffle_base.stl"
+                    scale="${base_mesh_scale_x} ${base_mesh_scale_y} ${base_mesh_scale_z}" />
+            </geometry>
+            <origin xyz="0 0 ${base_mesh_z_offset}" rpy="0 0 0" />
+            <material name="blue" />
+        </visual>
+        <collision>
+            <geometry>
                 <box size="${base_length} ${base_width} ${base_height}" />
             </geometry>
-            <!-- Raise the visual by half its height so the link frame is at ground level. -->
             <origin xyz="0 0 ${base_height / 2}" rpy="0 0 0" />
-            <material name="blue" />
-        </visual>
+        </collision>
     </link>
     <!-- Drive wheels: cylinders are rotated so their axles align with the Y-axis. -->
